File: pedai-hw.kicad_pcb (KiCad board)
At the start: 2 copper layers, 49 parts, among them J10 Conn_01x06, J11 Conn_01x16, J12 Conn_01x16, J13 Conn_01x08, J14 Conn_01x08, J15 Spare_ADC, J16 left_connector_blackpill, J17 right_connector_blackpill, J3 I2S_module, J4 Unused_pins_I2S, J5 LCD1602a, J6 Conn_01x06, J7 Conn_01x06, J8 Conn_01x06, J9 Conn_01x06

Commit message: fix: replaced 16 channel mux modules with 8 channels mux chips schematic concluded and added 3d models
Parts:
- removed J11, J12: Conn_01x16, Connector_PinSocket_2.54mm:PinSocket_1x16_P2.54mm_Vertical
- removed J13, J14: Conn_01x08, Connector_PinSocket_2.54mm:PinSocket_1x08_P2.54mm_Vertical
- removed J4: Unused_pins_I2S, Connector_PinSocket_2.54mm:PinSocket_1x09_P2.54mm_Vertical
- added D1: LED, LED_THT:LED_D3.0mm, F.Cu at (138.1, 96.4)
- added D2: LED, LED_THT:LED_D3.0mm, F.Cu at (138.1, 101.9)
- added IC1: CD4051BE, Library:CD4051BE, F.Cu at (83.5, 68.4)
- added IC2: CD4051BE, Library:CD4051BE, F.Cu at (122.5, 68.7)
- added IC3: CD4051BE, Library:CD4051BE, F.Cu at (152.8, 68.2)
- added IC4: CD4051BE, Library:CD4051BE, F.Cu at (184.3, 69.2)
- added IC5: CD4051BE, Library:CD4051BE, F.Cu at (216.5, 68.2)
- added IC6: CD4051BE, Library:CD4051BE, F.Cu at (254.7, 69.1)
- added J1: Conn_01x06, Connector_JST:JST_XH_B6B-XH-A_1x06_P2.50mm_Vertical, F.Cu at (260.0, 28.8)
- added R31: 150, Resistor_THT:R_Axial_DIN0204_L3.6mm_D1.6mm_P5.08mm_Vertical, F.Cu at (143.9, 95.2)
- added R32: 150, Resistor_THT:R_Axial_DIN0204_L3.6mm_D1.6mm_P5.08mm_Vertical, F.Cu at (143.9, 98.4)
- added R35: 1k, Resistor_THT:R_Axial_DIN0204_L3.6mm_D1.6mm_P5.08mm_Vertical, F.Cu at (261.0, 42.5)
- added R36: 1k, Resistor_THT:R_Axial_DIN0204_L3.6mm_D1.6mm_P5.08mm_Vertical, F.Cu at (257.9, 42.5)
- added R37: 1k, Resistor_THT:R_Axial_DIN0204_L3.6mm_D1.6mm_P5.08mm_Vertical, F.Cu at (254.7, 42.5)
- added R38: 1k, Resistor_THT:R_Axial_DIN0204_L3.6mm_D1.6mm_P5.08mm_Vertical, F.Cu at (251.6, 42.5)
- added R39: 1k, Resistor_THT:R_Axial_DIN0204_L3.6mm_D1.6mm_P5.08mm_Vertical, F.Cu at (248.4, 42.5)
- added R40: 1k, Resistor_THT:R_Axial_DIN0204_L3.6mm_D1.6mm_P5.08mm_Vertical, F.Cu at (245.2, 42.5)
- moved J15 73.8 mm to (167.0, 112.3), turned to 180 degrees
- moved J17 50.6 mm to (180.8, 137.8), turned to 180 degrees
- moved J3 47.0 mm to (123.9, 127.3)
- moved J5 34.8 mm to (225.2, 99.8), turned to 0 degrees
- moved J16 30.7 mm to (195.8, 137.8), turned to 180 degrees
- moved R33 27.1 mm to (213.8, 91.5), turned to 0 degrees
- moved R34 21.8 mm to (213.8, 102.0)
Connections:
- J16 pad 12: unconnected-(J16-Pin_12-Pad12) -> /MUX6_DATA
- J16 pad 14: /MUX_D0 -> /MUX1_DATA
- J16 pad 15: /MUX_D1 -> /MUX2_DATA
- J16 pad 16: unconnected-(J16-Pin_16-Pad16) -> /MUX5_DATA
- J16 pad 17: unconnected-(J16-Pin_17-Pad17) -> /MUX4_DATA
- J16 pad 7: /MUX_C0 -> /MUX3_DATA
- J17 pad 10: /MUX_C3 -> /MUX_C2
- J17 pad 17: unconnected-(J17-Pin_17-Pad17) -> /LED_SOUND
- J17 pad 18: unconnected-(J17-Pin_18-Pad18) -> /LED_MIDI
- J17 pad 8: /MUX_C1 -> /MUX_C0
- J17 pad 9: /MUX_C2 -> /MUX_C1

Commit message: WIP: layout work in progress
Parts:
- removed the R31 at (210.2, 40.9)
- removed the R32 at (207.0, 40.9)
- moved R25 174.8 mm to (66.0, 104.0), turned to 90 degrees
- moved J10 173.0 mm to (74.0, 113.5), turned to 0 degrees
- moved R35 172.2 mm to (100.2, 104.2), turned to 90 degrees
- moved J1 172.2 mm to (110.0, 113.2), turned to 0 degrees
- moved R26 166.8 mm to (71.5, 104.0), turned to 90 degrees
- moved R36 163.7 mm to (106.2, 104.2), turned to 90 degrees
- moved R27 158.8 mm to (77.0, 104.0), turned to 90 degrees
- moved R37 155.5 mm to (112.0, 104.2), turned to 90 degrees
- moved R28 150.9 mm to (82.5, 104.0), turned to 90 degrees
- moved R38 147.5 mm to (117.8, 104.5), turned to 90 degrees
- moved IC6 141.4 mm to (114.2, 85.4), turned to 180 degrees
- moved R29 141.0 mm to (88.0, 99.0)
- moved R39 139.5 mm to (123.5, 104.7), turned to 90 degrees
- moved IC5 137.4 mm to (80.2, 85.1), turned to 180 degrees
- moved R30 133.1 mm to (93.5, 99.0)
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
Commit message: layout and routing finished
Parts:
- added H1: MountingHole, MountingHole:MountingHole_4.3mm_M4, F.Cu at (202.5, 32.5)
- added H2: MountingHole, MountingHole:MountingHole_4.3mm_M4, F.Cu at (202.5, 127.5)
- added H3: MountingHole, MountingHole:MountingHole_4.3mm_M4, F.Cu at (57.5, 32.5)
- added H4: MountingHole, MountingHole:MountingHole_4.3mm_M4, F.Cu at (57.5, 127.5)
- R1, R10, R11, R12, R13, R14, R15, R16, R17, R18, R19, R2, R20, R21, R22, R23, R24, R25, R26, R27, R28, R29, R3, R30, R31, R32, R33, R34, R35, R36, R37, R38, R39, R4, R40, R5, R6, R7, R8, R9: footprint Resistor_THT:R_Axial_DIN0204_L3.6mm_D1.6mm_P5.08mm_Vertical -> Resistor_THT:R_Axial_DIN0204_L3.6mm_D1.6mm_P5.08mm_Horizontal
- moved R19 43.9 mm to (162.0, 58.7)
- moved R23 38.5 mm to (141.5, 49.8)
- moved R13 38.0 mm to (133.7, 58.2)
- moved R24 37.7 mm to (141.5, 60.0)
- moved J9 36.1 mm to (158.5, 41.0)
- moved R22 35.6 mm to (162.0, 67.0)
- moved R20 35.3 mm to (162.0, 50.2)
- moved IC4 35.1 mm to (151.7, 62.4)
- moved R21 33.5 mm to (157.6, 48.5), turned to 180 degrees
- moved R38 33.3 mm to (90.2, 85.8)
- moved R16 31.9 mm to (133.7, 66.7)
- moved R18 29.5 mm to (115.7, 58.4)
- moved R14 29.1 mm to (133.7, 49.7)
- moved R17 29.0 mm to (116.0, 48.2)
- moved J8 28.8 mm to (131.5, 41.0)
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Connections:
- J17 pad 1: +5V -> unconnected-(J17-Pin_1-Pad1)
Routing:
- net GND: track 0.00 -> 344.6 mm, vias 0 -> 2
- net /MUX_C0: track 0.00 -> 181.6 mm, vias 0 -> 1
- net /MUX_C1: track 0.00 -> 163.5 mm, vias 0 -> 3
- net /MUX_C2: track 0.00 -> 144.2 mm, vias 0 -> 3
- net /MUX1_DATA: track 0.00 -> 115.1 mm, vias 0 -> 3
- net /MUX5_DATA: track 0.00 -> 109.5 mm, vias 0 -> 1
- net /LCD_RS: track 0.00 -> 103.1 mm
- net /I2S_WS: track 0.00 -> 102.4 mm
- net /I2S_CLK: track 0.00 -> 99.4 mm, vias 0 -> 2
- net /I2S_SD: track 0.00 -> 98.7 mm, vias 0 -> 2
- net /LCD_ENABLE: track 0.00 -> 98.6 mm, vias 0 -> 2
- net /LCD_D0: track 0.00 -> 95.0 mm, vias 0 -> 2
- net /MUX2_DATA: track 0.00 -> 91.8 mm, vias 0 -> 1
- net /LCD_D1: track 0.00 -> 90.8 mm, vias 0 -> 2
- net /MUX6_DATA: track 0.00 -> 83.9 mm, vias 0 -> 1
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- added copper zone on B.Cu, net +3.3V
Other:
- board outline added: 160 x 110 mm

Commit message: fabrication output, silkscreen
Parts:
- removed H3, H4: MountingHole, MountingHole:MountingHole_4.3mm_M4
- moved H1 162.8 mm to (82.5, 142.5)
- moved H2 70.2 mm to (197.5, 57.5)
- moved D1 24.4 mm to (141.0, 106.0)
- moved D2 24.4 mm to (141.2, 97.0)
- moved R17 24.4 mm to (136.0, 62.2)
- moved R18 24.4 mm to (135.7, 72.4)
- moved IC1 24.4 mm to (93.2, 77.5)
- moved IC4 24.4 mm to (171.7, 76.4)
- moved R1 24.4 mm to (102.8, 75.8)
- moved R24 24.4 mm to (161.5, 74.0)
- moved IC2 24.4 mm to (119.0, 77.4)
- moved IC3 24.4 mm to (145.4, 76.3)
- moved IC5 24.4 mm to (93.5, 104.6)
- moved IC6 24.4 mm to (119.5, 104.4)
- moved J1 24.4 mm to (112.8, 127.8)
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Other:
- board size 160 x 110 mm -> 130 x 100 mm
- board text added: "150"
- board text added: "B1 to F#1"
- board text added: "B2 to F#2"
- board text added: "B3 to F#3"
- board text added: "C1 to F1"
- board text added: "F2 to C2"
- board text added: "F3 to C3"
- board text added: "MIDI ON"
- board text added: "SOUND ON"

Commit message: VERSION 0.9 ready for production silkscreen meme and not meme, ground pad, potentiometer for volume control and switch to turn off the device
Parts:
- added G***: LOGO, image:logo, F.Cu at (149.0, 140.0)
- added R41: 1k, Resistor_THT:R_Axial_DIN0204_L3.6mm_D1.6mm_P5.08mm_Horizontal, F.Cu at (80.7, 134.4)
- added RV1: R_Potentiometer, Potentiometer_THT:Potentiometer_Alps_RK163_Single_Horizontal, F.Cu at (114.6, 142.4)
- added SW1: SW_DIP_x01, Library:KCD1-101, F.Cu at (91.2, 144.0)
Connections:
- J15 pad 1: /SPARE_ADC_4 -> GND
- J15 pad 2: /SPARE_ADC_3 -> GND
- J17 pad 11: /SPARE_ADC_4 -> /VOLUME_CONTROL
- J17 pad 12: /SPARE_ADC_3 -> /SOUND_ON
Routing:
- net /SOUND_ON: track 0.00 -> 90.8 mm, vias 0 -> 2
- net GND: track 344.6 -> 414.3 mm
- net /VOLUME_CONTROL: track 0.00 -> 57.1 mm, vias 0 -> 1
- net /SPARE_ADC_3: track 12.3 -> 0.00 mm
- net /SPARE_ADC_4: track 12.3 -> 0.00 mm
- net /I2S_WS: track 102.4 -> 102.9 mm
- added copper zone on F.Cu, net GND
Other:
- board text added: "ADC1"
- board text added: "ADC2"
- board text added: "E ghe semo ancor, n'altro brusao?"
- board text added: "GND"
- board text added: "L'è 'na pedaliera speciale la fa do note per pedale"
- board text added: "PEDAI"
- board text added: "Pronto a la rozaa?"
- board text added: "Version 0.96 by gmazzucchi"
- board text added: "nuuumero 2"
- board text added: "nuuumero 3"
- board text added: "nuuumero 4"
- board text added: "nuuumero 5"
- board text added: "nuuumero 6"
- board text added: "nuuumero uuuuuuno (cit. Coca)"
- board text added: "tachete al graund"
- board text added: "values ad libitum"

Commit message: BREAKING: production
Parts:
- added C7: 100n, Capacitor_THT:CP_Radial_D4.0mm_P2.00mm, F.Cu at (190.5, 144.5)
- added J11: Conn_01x09, Connector_PinSocket_2.54mm:PinSocket_1x09_P2.54mm_Vertical, F.Cu at (160.5, 134.2)
- added J2: Ground connector 1, Connector_PinHeader_2.54mm:PinHeader_1x04_P2.54mm_Vertical, F.Cu at (190.1, 66.2)
- added J4: Ground connector 2, Connector_PinHeader_2.54mm:PinHeader_1x04_P2.54mm_Vertical, F.Cu at (190.1, 71.5)
- G***: moved to B.Cu
- moved G*** 18.1 mm to (141.5, 123.5), turned to 180 degrees
Connections:
- J5 pad 12: +5V -> GND
Routing:
- net GND: track 414.3 -> 458.6 mm, vias 2 -> 3
- net /I2S_WS: track 102.9 -> 108.2 mm
- net +5V: track 78.8 -> 83.2 mm
- net /key_inputs/NOTE_B3: track 32.9 -> 34.2 mm
- removed copper zone on F.Cu, net GND
