File: pedai-hw.kicad_pcb (KiCad board)
At the start: 2 copper layers, 710 x 70 mm, 31 parts, among them IC1 CD4051BQPWRQ1, IC2 CD4051BQPWRQ1, IC3 CD4051BQPWRQ1, J1 Conn_01x03, J10 Conn_01x01, J11 Conn_01x01, J12 Conn_01x01, J13 Conn_01x01, J14 Conn_01x01, J15 Conn_01x01, J16 left_connector_blackpill, J17 right_connector_blackpill, J18 Conn_01x01, J19 Conn_01x01, J2 Conn_01x01, J20 Conn_01x01, J21 Conn_01x01, J22 Conn_01x01, J23 Conn_01x01, J24 Conn_01x01, J25 Conn_01x01, J26 Conn_01x01, J27 Conn_01x01, J28 Conn_01x01, J3 Conn_01x01, J4 Conn_01x01, J5 Conn_01x01, J6 Conn_01x01, J7 Conn_01x01, J8 Conn_01x01, J9 Conn_01x01

Commit message: board is almost ready for production still looking for mistakes and inaccuracies
Signed-off-by: gmazzucchi <giacomo.mazzucchi@protonmail.com>
Parts:
- added H1: MountingHole, MountingHole:MountingHole_4.3mm_M4, F.Cu at (64.2, 277.2)
- added H2: MountingHole, MountingHole:MountingHole_4.3mm_M4, F.Cu at (786.2, 277.2)
- added J29: Conn_01x01, Connector_Wire:SolderWirePad_1x01_SMD_5x10mm, F.Cu at (763.8, 282.0)
- added R1: 1000, Resistor_SMD:R_1206_3216Metric, F.Cu at (287.0, 280.8)
- added R2: 1000, Resistor_SMD:R_1206_3216Metric, F.Cu at (755.7, 274.8)
- added R3: 1000, Resistor_SMD:R_1206_3216Metric, F.Cu at (513.1, 273.0)
- IC1, IC2, IC3: moved to F.Cu
- moved IC1 455.0 mm to (287.2, 274.2)
- moved J25 262.7 mm to (675.0, 277.5)
- moved IC3 262.1 mm to (513.1, 279.5), turned to 0 degrees
- moved J24 261.1 mm to (650.0, 277.5)
- moved J21 259.9 mm to (575.0, 277.5)
- moved J23 259.1 mm to (625.5, 277.5)
- moved J22 257.0 mm to (600.0, 277.0)
- moved J28 250.4 mm to (775.0, 277.5)
- moved J26 247.0 mm to (700.0, 277.5)
- moved J27 238.1 mm to (725.0, 277.5)
- moved J20 233.5 mm to (524.5, 277.5)
- moved J19 232.2 mm to (500.0, 277.5)
- moved J18 226.4 mm to (474.5, 277.5)
- moved J14 222.5 mm to (425.0, 277.0)
- moved J15 218.2 mm to (449.5, 277.0)
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Connections:
- J16 pad 18: +3.3V -> unconnected-(J16-Pin_18-Pad18)
- J16 pad 20: unconnected-(J16-Pin_20-Pad20) -> +3.3V
- J17 pad 2: GND -> unconnected-(J17-Pin_2-Pad2)
Routing:
- net GND: track 0.00 -> 534.4 mm, vias 0 -> 8
- net /MUX_C2: track 0.00 -> 519.6 mm, vias 0 -> 7
- net /MUX_C3: track 0.00 -> 514.0 mm, vias 0 -> 6
- net +3.3V: track 0.00 -> 513.2 mm, vias 0 -> 8
- net /MUX_C1: track 0.00 -> 512.7 mm, vias 0 -> 7
- net /MUX_D1: track 0.00 -> 492.6 mm, vias 0 -> 4
- net /MUX_D3: track 0.00 -> 290.2 mm, vias 0 -> 4
- net /NOTE_8: track 0.00 -> 230.1 mm, vias 0 -> 2
- net /NOTE_16: track 0.00 -> 228.8 mm, vias 0 -> 3
- net /NOTE_0: track 0.00 -> 213.7 mm
- net /NOTE_9: track 0.00 -> 206.7 mm, vias 0 -> 2
- net /NOTE_1: track 0.00 -> 188.1 mm
- net /NOTE_10: track 0.00 -> 183.5 mm, vias 0 -> 2
- net /NOTE_17: track 0.00 -> 178.3 mm, vias 0 -> 2
- net /NOTE_11: track 0.00 -> 166.0 mm, vias 0 -> 4
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Other:
- board size 710 x 70 mm -> 734.5 x 70 mm

Commit message: fix: removed multiplexer and attached directly to GPIOs fix: removed I2S interface for sound feat: added a UART to communicate with the mainboard
Parts:
- removed IC1, IC2, IC3: CD4051BQPWRQ1, pedalinator_library:CD4051BQ
- removed J1: Conn_01x03, Connector_PinHeader_2.00mm:PinHeader_1x03_P2.00mm_Vertical
- added J30: Conn_01x02, Connector_PinSocket_2.54mm:PinSocket_1x02_P2.54mm_Vertical, F.Cu at (749.1, 217.4)
- added R10: 1k, Resistor_THT:R_Axial_DIN0207_L6.3mm_D2.5mm_P10.16mm_Horizontal, F.Cu at (338.0, 273.6)
- added R11: 1k, Resistor_THT:R_Axial_DIN0207_L6.3mm_D2.5mm_P10.16mm_Horizontal, F.Cu at (363.0, 273.7)
- added R12: 1k, Resistor_THT:R_Axial_DIN0207_L6.3mm_D2.5mm_P10.16mm_Horizontal, F.Cu at (387.9, 274.0)
- added R13: 1k, Resistor_THT:R_Axial_DIN0207_L6.3mm_D2.5mm_P10.16mm_Horizontal, F.Cu at (438.0, 274.0)
- added R14: 1k, Resistor_THT:R_Axial_DIN0207_L6.3mm_D2.5mm_P10.16mm_Horizontal, F.Cu at (462.5, 274.0)
- added R15: 1k, Resistor_THT:R_Axial_DIN0207_L6.3mm_D2.5mm_P10.16mm_Horizontal, F.Cu at (487.5, 274.0)
- added R16: 1k, Resistor_THT:R_Axial_DIN0207_L6.3mm_D2.5mm_P10.16mm_Horizontal, F.Cu at (513.0, 274.0)
- added R17: 1k, Resistor_THT:R_Axial_DIN0207_L6.3mm_D2.5mm_P10.16mm_Horizontal, F.Cu at (537.5, 274.0)
- added R18: 1k, Resistor_THT:R_Axial_DIN0207_L6.3mm_D2.5mm_P10.16mm_Horizontal, F.Cu at (587.9, 274.0)
- added R19: 1k, Resistor_THT:R_Axial_DIN0207_L6.3mm_D2.5mm_P10.16mm_Horizontal, F.Cu at (612.9, 274.2)
- added R20: 1k, Resistor_THT:R_Axial_DIN0207_L6.3mm_D2.5mm_P10.16mm_Horizontal, F.Cu at (638.3, 274.2)
- added R21: 1k, Resistor_THT:R_Axial_DIN0207_L6.3mm_D2.5mm_P10.16mm_Horizontal, F.Cu at (662.9, 274.2)
- added R22: 1k, Resistor_THT:R_Axial_DIN0207_L6.3mm_D2.5mm_P10.16mm_Horizontal, F.Cu at (688.0, 274.0)
- added R23: 1k, Resistor_THT:R_Axial_DIN0207_L6.3mm_D2.5mm_P10.16mm_Horizontal, F.Cu at (712.9, 274.0)
- added R24: 1k, Resistor_THT:R_Axial_DIN0207_L6.3mm_D2.5mm_P10.16mm_Horizontal, F.Cu at (737.8, 274.0)
- added R25: 1k, Resistor_THT:R_Axial_DIN0207_L6.3mm_D2.5mm_P10.16mm_Horizontal, F.Cu at (758.6, 273.8)
- added R4: 1k, Resistor_THT:R_Axial_DIN0207_L6.3mm_D2.5mm_P10.16mm_Horizontal, F.Cu at (163.0, 273.0)
- added R5: 1k, Resistor_THT:R_Axial_DIN0207_L6.3mm_D2.5mm_P10.16mm_Horizontal, F.Cu at (188.1, 273.0)
- added R6: 1k, Resistor_THT:R_Axial_DIN0207_L6.3mm_D2.5mm_P10.16mm_Horizontal, F.Cu at (238.0, 273.6)
- added R7: 1k, Resistor_THT:R_Axial_DIN0207_L6.3mm_D2.5mm_P10.16mm_Horizontal, F.Cu at (263.3, 273.4)
- added R8: 1k, Resistor_THT:R_Axial_DIN0207_L6.3mm_D2.5mm_P10.16mm_Horizontal, F.Cu at (288.0, 273.6)
- added R9: 1k, Resistor_THT:R_Axial_DIN0207_L6.3mm_D2.5mm_P10.16mm_Horizontal, F.Cu at (313.0, 273.6)
- R1, R2, R3: value 1000 -> 1k; footprint Resistor_SMD:R_1206_3216Metric -> Resistor_THT:R_Axial_DIN0207_L6.3mm_D2.5mm_P10.16mm_Horizontal
- moved R2 642.5 mm to (113.2, 273.0), turned to 180 degrees
- moved R3 375.1 mm to (138.0, 273.0)
- moved R1 199.0 mm to (88.2, 273.0), turned to 180 degrees
- moved J22 0.60 mm to (600.0, 277.6)
- moved J12 0.50 mm to (350.0, 277.0)
- moved J14 0.40 mm to (425.0, 277.4)
- moved J15 0.40 mm to (449.5, 277.4)
- moved J23 0.10 mm to (625.5, 277.6)
- moved J24 0.10 mm to (650.0, 277.6)
Connections:
- J10 pad 1: /NOTE_8 -> /NOTE_9
- J11 pad 1: /NOTE_9 -> /NOTE_10
- J12 pad 1: /NOTE_10 -> /NOTE_11
- J13 pad 1: /NOTE_11 -> /NOTE_12
- J14 pad 1: /NOTE_12 -> /NOTE_13
- J15 pad 1: /NOTE_13 -> /NOTE_14
- J16 pad 1: unconnected-(J16-Pin_1-Pad1) -> /NOTE_22
- J16 pad 10: unconnected-(J16-Pin_10-Pad10) -> /NOTE_10
- J16 pad 11: /NOTE_24 -> /NOTE_14
- J16 pad 12: /MUX_D3 -> /NOTE_15
- J16 pad 13: /MUX_D2 -> /NOTE_16
- J16 pad 14: /MUX_D1 -> /NOTE_17
- J16 pad 15: /MUX_C3 -> /NOTE_18
- J16 pad 16: /MUX_C2 -> /NOTE_19
- J16 pad 17: /MUX_C1 -> /NOTE_20
- J16 pad 2: unconnected-(J16-Pin_2-Pad2) -> /NOTE_23
- J16 pad 3: unconnected-(J16-Pin_3-Pad3) -> /NOTE_24
- J16 pad 4: unconnected-(J16-Pin_4-Pad4) -> /NOTE_25
- J16 pad 5: unconnected-(J16-Pin_5-Pad5) -> /NOTE_9
- J16 pad 6: unconnected-(J16-Pin_6-Pad6) -> /UART_TX
- J16 pad 7: unconnected-(J16-Pin_7-Pad7) -> /UART_RX
- J17 pad 10: unconnected-(J17-Pin_10-Pad10) -> /NOTE_6
- J17 pad 11: /I2S_WS -> /NOTE_5
- J17 pad 12: unconnected-(J17-Pin_12-Pad12) -> /NOTE_4
- J17 pad 13: unconnected-(J17-Pin_13-Pad13) -> /NOTE_3
- J17 pad 14: unconnected-(J17-Pin_14-Pad14) -> /NOTE_2
- J17 pad 15: unconnected-(J17-Pin_15-Pad15) -> /NOTE_1
- J17 pad 4: unconnected-(J17-Pin_4-Pad4) -> /NOTE_21
- J17 pad 5: unconnected-(J17-Pin_5-Pad5) -> /NOTE_13
- J17 pad 6: unconnected-(J17-Pin_6-Pad6) -> /NOTE_12
- J17 pad 7: unconnected-(J17-Pin_7-Pad7) -> /NOTE_11
- J17 pad 8: /I2S_SD -> /NOTE_8
- J17 pad 9: /I2S_CK -> /NOTE_7
- J18 pad 1: /NOTE_14 -> /NOTE_15
- J19 pad 1: /NOTE_15 -> /NOTE_16
- J2 pad 1: /NOTE_0 -> /NOTE_1
- J20 pad 1: /NOTE_16 -> /NOTE_17
- J21 pad 1: /NOTE_17 -> /NOTE_18
- J22 pad 1: /NOTE_18 -> /NOTE_19
- J23 pad 1: /NOTE_19 -> /NOTE_20
- J24 pad 1: /NOTE_20 -> /NOTE_21
- J25 pad 1: /NOTE_21 -> /NOTE_22
- J26 pad 1: /NOTE_22 -> /NOTE_23
- J27 pad 1: /NOTE_23 -> /NOTE_24
- J28 pad 1: /NOTE_24 -> /NOTE_25
- J3 pad 1: /NOTE_1 -> /NOTE_2
- J4 pad 1: /NOTE_2 -> /NOTE_3
- J5 pad 1: /NOTE_3 -> /NOTE_4
- J6 pad 1: /NOTE_4 -> /NOTE_5
- J7 pad 1: /NOTE_5 -> /NOTE_6
- J8 pad 1: /NOTE_6 -> /NOTE_7
- J9 pad 1: /NOTE_7 -> /NOTE_8
- R1 pad 2: /MUX_D1 -> /NOTE_1
- R2 pad 2: /MUX_D2 -> /NOTE_2
- R3 pad 2: /MUX_D3 -> /NOTE_3
Routing:
- net /NOTE_6: track 49.5 -> 585.9 mm, vias 2 -> 1
- net /NOTE_7: track 22.6 -> 555.9 mm, vias 2 -> 1
- net /NOTE_5: track 82.1 -> 612.3 mm, vias 2 -> 1
- net /NOTE_3: track 137.1 -> 657.8 mm, vias 2 -> 1
- net /MUX_C2: track 519.6 -> 0.00 mm, vias 7 -> 0
- net /NOTE_2: track 162.6 -> 680.4 mm, vias 0 -> 1
- net /NOTE_1: track 188.1 -> 703.2 mm, vias 0 -> 1
- net /MUX_C3: track 514.0 -> 0.00 mm, vias 6 -> 0
- net /MUX_C1: track 512.7 -> 0.00 mm, vias 7 -> 0
- net /NOTE_4: track 134.0 -> 635.2 mm, vias 2 -> 1
- net GND: track 534.4 -> 34.7 mm, vias 8 -> 1
- net /MUX_D1: track 492.6 -> 0.00 mm, vias 4 -> 0
- net /NOTE_12: track 87.7 -> 439.3 mm, vias 0 -> 2
- net /NOTE_13: track 61.8 -> 388.7 mm, vias 0 -> 2
- net /NOTE_14: track 38.3 -> 354.6 mm, vias 0 -> 1
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
Commit message: production
Parts:
- added C1: 10u, Capacitor_SMD:C_0603_1608Metric, F.Cu at (748.8, 265.6)
- added C2: 100n, Capacitor_SMD:C_0603_1608Metric, F.Cu at (745.5, 265.6)
- added C3: 220u, Capacitor_SMD:C_0603_1608Metric, F.Cu at (752.0, 265.6)
- added H3: MountingHole, MountingHole:MountingHole_3.2mm_M3_Pad, F.Cu at (203.5, 277.8)
- added H4: MountingHole, MountingHole:MountingHole_3.2mm_M3_Pad, F.Cu at (406.4, 276.6)
- added H5: MountingHole, MountingHole:MountingHole_3.2mm_M3_Pad, F.Cu at (554.4, 276.2)
- H1, H2: footprint MountingHole:MountingHole_4.3mm_M4 -> MountingHole:MountingHole_3.2mm_M3_Pad
- J30: footprint Connector_PinSocket_2.54mm:PinSocket_1x02_P2.54mm_Vertical -> Connector_PinHeader_2.54mm:PinHeader_1x04_P2.54mm_Vertical
- R1, R10, R11, R12, R13, R14, R15, R16, R17, R18, R19, R2, R20, R21, R22, R23, R24, R25, R3, R4, R5, R6, R7, R8, R9: value 1k -> 4.7k
- moved J30 2.65 mm to (746.4, 217.4)
Routing:
- net +3.3V: track 700.8 -> 764.9 mm, vias 0 -> 1
- net GND: track 34.7 -> 94.9 mm, vias 1 -> 2
- net /NOTE_8: track 532.3 -> 536.2 mm
- net /NOTE_14: track 354.6 -> 352.4 mm
- net /UART_RX: track 21.3 -> 20.2 mm
Other:
- outline, holes or cut-outs redrawn
